File: tools/backplane/pcb/backplane.kicad_pcb (KiCad board)
At the start: 0 parts

Commit message: start adding connectors to the backplane
Parts:
- added J1: 09032967825, 09032967825:09032967825, F.Cu at (20.6, 16.2)
- added J10: 09032967825, 09032967825:09032967825, F.Cu at (0.30, 16.2)
- added J2: 09032967825, 09032967825:09032967825, F.Cu at (40.9, 16.2)
- added J3: 09032967825, 09032967825:09032967825, F.Cu at (61.3, 16.2)
- added J4: 09032967825, 09032967825:09032967825, F.Cu at (81.6, 16.2)
- added J5: 09032967825, 09032967825:09032967825, F.Cu at (101.9, 16.2)
- added J6: 09032967825, 09032967825:09032967825, F.Cu at (122.2, 16.2)
- added J7: 09032967825, 09032967825:09032967825, F.Cu at (142.5, 16.2)
- added J8: 09032967825, 09032967825:09032967825, F.Cu at (162.9, 16.2)
- added J9: 09032967825, 09032967825:09032967825, F.Cu at (183.2, 16.2)
- added REF**: MountingHole_2.7mm, MountingHole:MountingHole_2.7mm, F.Cu at (20.3, 0.00)
- added REF**: MountingHole_2.7mm, MountingHole:MountingHole_2.7mm, F.Cu at (40.6, 122.5)
- added REF**: MountingHole_2.7mm, MountingHole:MountingHole_2.7mm, F.Cu at (121.9, 0.00)
- added REF**: MountingHole_2.7mm, MountingHole:MountingHole_2.7mm, F.Cu at (61.0, 0.00)
- added REF**: MountingHole_2.7mm, MountingHole:MountingHole_2.7mm, F.Cu at (121.9, 122.5)
- added REF**: MountingHole_2.7mm, MountingHole:MountingHole_2.7mm, F.Cu at (61.0, 122.5)
- added REF**: MountingHole_2.7mm, MountingHole:MountingHole_2.7mm, F.Cu at (81.3, 0.00)
- added REF**: MountingHole_2.7mm, MountingHole:MountingHole_2.7mm, F.Cu at (142.2, 122.5)
- added REF**: MountingHole_2.7mm, MountingHole:MountingHole_2.7mm, F.Cu at (81.3, 122.5)
- added REF**: MountingHole_2.7mm, MountingHole:MountingHole_2.7mm, F.Cu at (101.6, 0.00)
- added REF**: MountingHole_2.7mm, MountingHole:MountingHole_2.7mm, F.Cu at (142.2, 0.00)
- added REF**: MountingHole_2.7mm, MountingHole:MountingHole_2.7mm, F.Cu at (162.6, 0.00)
- added REF**: MountingHole_2.7mm, MountingHole:MountingHole_2.7mm, F.Cu at (40.6, 0.00)
- added REF**: MountingHole_2.7mm, MountingHole:MountingHole_2.7mm, F.Cu at (182.9, 122.5)
- added REF**: MountingHole_2.7mm, MountingHole:MountingHole_2.7mm, F.Cu at (0.00, 0.00)
- added REF**: MountingHole_2.7mm, MountingHole:MountingHole_2.7mm, F.Cu at (101.6, 122.5)
- added REF**: MountingHole_2.7mm, MountingHole:MountingHole_2.7mm, F.Cu at (0.00, 122.5)
- added REF**: MountingHole_2.7mm, MountingHole:MountingHole_2.7mm, F.Cu at (162.6, 122.5)
- added REF**: MountingHole_2.7mm, MountingHole:MountingHole_2.7mm, F.Cu at (20.3, 122.5)
- added REF**: MountingHole_2.7mm, MountingHole:MountingHole_2.7mm, F.Cu at (182.9, 0.00)
Other:
- copper layers 0 -> 2
